Commit message: Name changing

File: urdf/robotiq_c2_model.urdf (robot description, URDF)
Before this commit: robot robotiq_c2_model, 10 links, 9 joints
Links:
- link robotiq_85_adapter_link: geometry collision mesh filename=package://robotiq_c2_description/meshes/robotiq_c2/collisio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; visual mesh filename=package://robotiq_c2_description/meshes/robotiq_c2/visual/r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
- link robotiq_85_base_link: geometry collision mesh filename=package://robotiq_c2_description/meshes/robotiq_c2/collisio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; visual mesh filename=package://robotiq_c2_description/meshes/robotiq_c2/visual/r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
- link robotiq_85_left_finger_link: geometry collision mesh filename=package://robotiq_c2_description/meshes/robotiq_c2/collisio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; visual mesh filename=package://robotiq_c2_description/meshes/robotiq_c2/visual/r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
- link robotiq_85_left_finger_tip_link: geometry collision mesh filename=package://robotiq_c2_description/meshes/robotiq_c2/collisio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; visual mesh filename=package://robotiq_c2_description/meshes/robotiq_c2/visual/r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
- link robotiq_85_left_inner_knuckle_link: geometry collision mesh filename=package://robotiq_c2_description/meshes/robotiq_c2/collisio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; visual mesh filename=package://robotiq_c2_description/meshes/robotiq_c2/visual/r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
- link robotiq_85_left_knuckle_link: geometry collision mesh filename=package://robotiq_c2_description/meshes/robotiq_c2/collisio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; visual mesh filename=package://robotiq_c2_description/meshes/robotiq_c2/visual/r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
- link robotiq_85_right_finger_link: geometry collision mesh filename=package://robotiq_c2_description/meshes/robotiq_c2/collisio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; visual mesh filename=package://robotiq_c2_description/meshes/robotiq_c2/visual/r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
- link robotiq_85_right_finger_tip_link: geometry collision mesh filename=package://robotiq_c2_description/meshes/robotiq_c2/collisio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; visual mesh filename=package://robotiq_c2_description/meshes/robotiq_c2/visual/r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
- link robotiq_85_right_inner_knuckle_link: geometry collision mesh filename=package://robotiq_c2_description/meshes/robotiq_c2/collisio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; visual mesh filename=package://robotiq_c2_description/meshes/robotiq_c2/visual/r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
- link robotiq_85_right_knuckle_link: geometry collision mesh filename=package://robotiq_c2_description/meshes/robotiq_c2/collisio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; visual mesh filename=package://robotiq_c2_description/meshes/robotiq_c2/visual/r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

File: urdf/robotiq_c2_model.xacro (robot description, xacro)
@@ -5,5 +5,5 @@
  -->
 <robot name="robotiq_c2_model" xmlns:xacro="http://ros.org/wiki/xacro">
-    <xacro:include filename="$(find robotiq_c2_model_visualization)/urdf/robotiq_c2_model_macro.xacro" />
+    <xacro:include filename="$(find robotiq_c2_description)/urdf/robotiq_c2_model_macro.xacro" />
     <xacro:robotiq_c2_model prefix=""/>
 </robot>

File: urdf/robotiq_c2_model_macro.xacro (robot description, xacro)
@@ -7,5 +7,5 @@
 -->
 <robot xmlns:xacro="http://ros.org/wiki/xacro">
-<xacro:include filename="$(find robotiq_c2_model_visualization)/urdf/robotiq_c2_model.gazebo.xacro" />
+<xacro:include filename="$(find robotiq_c2_description)/urdf/robotiq_c2_model.gazebo.xacro" />
   <xacro:macro name="robotiq_c2_model" params="prefix parent *origin">
     <xacro:robotiq_c2_model_gazebo prefix="${prefix}"/>
@@ -21,5 +21,5 @@
     <visual>
       <geometry>
-        <mesh filename="package://robotiq_c2_model_visualization/meshes/robotiq_c2/visual/robotiq_85_gripper_base.dae"/>
+        <mesh filename="package://robotiq_c2_description/meshes/robotiq_c2/visual/robotiq_85_gripper_base.dae"/>
       </geometry>
       <origin rpy="3.1415 0 1.5707" xyz="0 0 0"/>
@@ -27,5 +27,5 @@
     <collision>
       <geometry>
-        <mesh filename="package://robotiq_c2_model_visualization/meshes/robotiq_c2/collision/robotiq_85_gripper_base.dae"/>
+        <mesh filename="package://robotiq_c2_description/meshes/robotiq_c2/collision/robotiq_85_gripper_base.dae"/>
       </geometry>
       <origin rpy="1.5707 0 1.5707" xyz="0 0 0"/>
@@ -61,5 +61,5 @@
     <visual>
       <geometry>
-        <mesh filename="package://robotiq_c2_model_visualization/meshes/robotiq_c2/visual/robotiq_85_gripper_joint_0_L.dae"/>
+        <mesh filename="package://robotiq_c2_description/meshes/robotiq_c2/visual/robotiq_85_gripper_joint_0_L.dae"/>
       </geometry>
       <origin rpy="3.14159 -1.5707 0" xyz="0 .04191 -.0306"/>
@@ -67,5 +67,5 @@
     <collision>
       <geometry>
-        <mesh filename="package://robotiq_c2_model_visualization/meshes/robotiq_c2/collision/robotiq_85_gripper_joint_0_L.dae"/>
+        <mesh filename="package://robotiq_c2_description/meshes/robotiq_c2/collision/robotiq_85_gripper_joint_0_L.dae"/>
       </geometry>
       <origin rpy="1.5707 -1.5707 0" xyz="0 .04191 -.0306"/>
@@ -82,5 +82,5 @@
     <visual>
       <geometry>
-        <mesh filename="package://robotiq_c2_model_visualization/meshes/robotiq_c2/visual/robotiq_85_gripper_joint_0_R.dae"/>
+        <mesh filename="package://robotiq_c2_description/meshes/robotiq_c2/visual/robotiq_85_gripper_joint_0_R.dae"/>
       </geometry>
       <origin rpy="3.14159 1.5707 0" xyz="0 .04191 -.0306"/>
@@ -88,5 +88,5 @@
     <collision>
       <geometry>
-        <mesh filename="package://robotiq_c2_model_visualization/meshes/robotiq_c2/collision/robotiq_85_gripper_joint_0_R.dae"/>
+        <mesh filename="package://robotiq_c2_description/meshes/robotiq_c2/collision/robotiq_85_gripper_joint_0_R.dae"/>
       </geometry>
       <origin rpy="1.5707 1.5707 0" xyz="0 .04191 -.0306"/>
@@ -121,5 +121,5 @@
     <visual>
       <geometry>
-        <mesh filename="package://robotiq_c2_model_visualization/meshes/robotiq_c2/visual/robotiq_85_gripper_joint_1_L.dae"/>
+        <mesh filename="package://robotiq_c2_description/meshes/robotiq_c2/visual/robotiq_85_gripper_joint_1_L.dae"/>
       </geometry>
       <origin rpy="0 1.5707 0" xyz="0 -.03683 .06194"/>
@@ -127,5 +127,5 @@
     <collision>
       <geometry>
-        <mesh filename="package://robotiq_c2_model_visualization/meshes/robotiq_c2/collision/robotiq_85_gripper_joint_1_L.dae"/>
+        <mesh filename="package://robotiq_c2_description/meshes/robotiq_c2/collision/robotiq_85_gripper_joint_1_L.dae"/>
       </geometry>
       <origin rpy="-1.5707 1.5707 0" xyz="0 -.03683 .06194"/>
@@ -142,5 +142,5 @@
     <visual>
       <geometry>
-        <mesh filename="package://robotiq_c2_model_visualization/meshes/robotiq_c2/visual/robotiq_85_gripper_joint_1_R.dae"/>
+        <mesh filename="package://robotiq_c2_description/meshes/robotiq_c2/visual/robotiq_85_gripper_joint_1_R.dae"/>
       </geometry>
       <origin rpy="0 -1.5707 0" xyz="0 -.03683 .06194"/>
@@ -148,5 +148,5 @@
     <collision>
       <geometry>
-        <mesh filename="package://robotiq_c2_model_visualization/meshes/robotiq_c2/collision/robotiq_85_gripper_joint_1_R.dae"/>
+        <mesh filename="package://robotiq_c2_description/meshes/robotiq_c2/collision/robotiq_85_gripper_joint_1_R.dae"/>
       </geometry>
       <origin rpy="-1.5707 -1.5707 0" xyz="0 -.03683 .06194"/>
@@ -183,5 +183,5 @@
     <visual>
       <geometry>
-        <mesh filename="package://robotiq_c2_model_visualization/meshes/robotiq_c2/visual/robotiq_85_gripper_joint_2_L.dae"/>
+        <mesh filename="package://robotiq_c2_description/meshes/robotiq_c2/visual/robotiq_85_gripper_joint_2_L.dae"/>
       </geometry>
       <origin rpy="0 1.5707 0" xyz="0 -.04843 .0127"/>
@@ -189,5 +189,5 @@
     <collision>
       <geometry>
-        <mesh filename="package://robotiq_c2_model_visualization/meshes/robotiq_c2/collision/robotiq_85_gripper_joint_2_L.dae"/>
+        <mesh filename="package://robotiq_c2_description/meshes/robotiq_c2/collision/robotiq_85_gripper_joint_2_L.dae"/>
       </geometry>
       <origin rpy="-1.5707 1.5707 0" xyz="0 -.04843 .0127"/>
@@ -204,5 +204,5 @@
     <visual>
       <geometry>
-        <mesh filename="package://robotiq_c2_model_visualization/meshes/robotiq_c2/visual/robotiq_85_gripper_joint_2_R.dae"/>
+        <mesh filename="package://robotiq_c2_description/meshes/robotiq_c2/visual/robotiq_85_gripper_joint_2_R.dae"/>
       </geometry>
       <origin rpy="0 -1.5707 0" xyz="0 -.04843 .0127"/>
@@ -210,5 +210,5 @@
     <collision>
       <geometry>
-        <mesh filename="package://robotiq_c2_model_visualization/meshes/robotiq_c2/collision/robotiq_85_gripper_joint_2_R.dae"/>
+        <mesh filename="package://robotiq_c2_description/meshes/robotiq_c2/collision/robotiq_85_gripper_joint_2_R.dae"/>
       </geometry>
       <origin rpy="-1.5707 -1.5707 0" xyz="0 -.04843 .0127"/>
@@ -245,5 +245,5 @@
     <visual>
       <geometry>
-        <mesh filename="package://robotiq_c2_model_visualization/meshes/robotiq_c2/visual/robotiq_85_gripper_joint_3_L.dae"/>
+        <mesh filename="package://robotiq_c2_description/meshes/robotiq_c2/visual/robotiq_85_gripper_joint_3_L.dae"/>
       </geometry>
       <origin rpy="0 1.5707 0" xyz="0 -.090381 .051505"/>
@@ -251,5 +251,5 @@
     <collision>
       <geometry>
-        <mesh filename="package://robotiq_c2_model_visualization/meshes/robotiq_c2/collision/robotiq_85_gripper_joint_3_L.dae"/>
+        <mesh filename="package://robotiq_c2_description/meshes/robotiq_c2/collision/robotiq_85_gripper_joint_3_L.dae"/>
       </geometry>
       <origin rpy="-1.5707 1.5707 0" xyz="0 -.090381 .051505"/>
@@ -266,5 +266,5 @@
     <visual>
       <geometry>
-        <mesh filename="package://robotiq_c2_model_visualization/meshes/robotiq_c2/visual/robotiq_85_gripper_joint_3_R.dae"/>
+        <mesh filename="package://robotiq_c2_description/meshes/robotiq_c2/visual/robotiq_85_gripper_joint_3_R.dae"/>
       </geometry>
       <origin rpy="0 -1.5707 0" xyz="0 -.090381 .051505"/>
@@ -272,5 +272,5 @@
     <collision>
       <geometry>
-        <mesh filename="package://robotiq_c2_model_visualization/meshes/robotiq_c2/collision/robotiq_85_gripper_joint_3_R.dae"/>
+        <mesh filename="package://robotiq_c2_description/meshes/robotiq_c2/collision/robotiq_85_gripper_joint_3_R.dae"/>
       </geometry>
       <origin rpy="-1.5707 -1.5707 0" xyz="0 -.090381 .051505"/>
